File: rev2/oibus-mini-CCC.kicad_pcb (KiCad board)
At the start: 2 copper layers, 37 x 60 mm, 91 parts, among them J1 Conn_01x04_Female, J2 USB_B_Micro, J3 uavcan_5pins, P1 TC2030-MCP, Q1 DMG3415U-7, Q2 NMOS, Q3 NMOS, SW1 SW_Push, SW2 SW_Push, U1 AP2112K-3.3, U10 TPD3E001DRLR, U2 SAM-M8Q, U3 NINA-B311-00B, U4 MCP73831-2-OT, U5 MCP1624T, U6 SHT31-DIS-B, U7 TCAN330, U8 STM32F303CCTx, U9 DW01C-G, Y1 16M, Y2 32kHz

Commit message: generated gerber V2
Other:
- outline, holes or cut-outs redrawn
- board text removed: "BLUETOOTH"
Changed lines of the file:
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@@
   (general
     (thickness 1.6)
-    (drawings 56)
+    (drawings 55)
     (tracks 1427)
     (zones 0)
@@
   (page A4)
   (layers
-    (0 F.Cu signal hide)
+    (0 F.Cu signal)
     (31 B.Cu signal hide)
     (32 B.Adhes user hide)
     (33 F.Adhes user hide)
     (35 F.Paste user hide)
-    (36 B.SilkS user hide)
+    (36 B.SilkS user)
     (37 F.SilkS user)
     (38 B.Mask user)
@@
     )
   )
+  (gr_arc (start 2.4 -18.4) (end 2.4 -18.8) (angle -180) (layer Edge.Cuts) (width 0.15))
+  (gr_arc (start 3.1 -23.2) (end 3.1 -23.6) (angle -180) (layer Edge.Cuts) (width 0.15))
+  (gr_arc (start 4.2 -20.8) (end 4.2 -18) (angle -180) (layer Edge.Cuts) (width 0.15))
   (gr_poly (pts (xy 0 -23) (xy 4.4 -23) (xy 5.8 -22.6) (xy 6.4 -21.2) (xy 6.4 -20.2) (xy 5.8 -19.2) (xy 4.6 -18.4) (xy 2.4 -18.4) (xy 0 -18.4)) (layer F.SilkS) (width 0.15))
   (gr_text PWR (at 4.55 -30 270) (layer F.SilkS)
@@
   )
   (gr_arc (start 4.2 -20.8) (end 4.2 -18.8) (angle -180) (layer Edge.Cuts) (width 0.15))
-  (gr_arc (start 2.3 -18.5) (end 2.3 -18.8) (angle -180) (layer Edge.Cuts) (width 0.15))
-  (gr_arc (start 3.1 -23.1) (end 3.1 -23.4) (angle -180) (layer Edge.Cuts) (width 0.15))
-  (gr_line (start 2.3 -18.2) (end 4.2 -18.2) (layer Edge.Cuts) (width 0.15))
+  (gr_line (start 2.3 -18) (end 4.2 -18) (layer Edge.Cuts) (width 0.15))
   (gr_line (start 4.2 -18.8) (end 2.3 -18.8) (layer Edge.Cuts) (width 0.15))
   (gr_line (start 3.1 -22.8) (end 4.2 -22.8) (layer Edge.Cuts) (width 0.15))
-  (gr_line (start 4.2 -23.4) (end 3.1 -23.4) (layer Edge.Cuts) (width 0.15))
-  (gr_arc (start 4.2 -20.8) (end 4.2 -18.2) (angle -180) (layer Edge.Cuts) (width 0.15))
+  (gr_line (start 4.2 -23.6) (end 3.1 -23.6) (layer Edge.Cuts) (width 0.15))
   (gr_text UART (at 2.5 -55.25) (layer B.SilkS)
     (effects (font (size 1 1) (thickness 0.2)) (justify mirror))
@@
     (effects (font (size 1 1) (thickness 0.2)) (justify mirror))
   )
-  (gr_text "BLUETOOTH\n" (at 36 -52.2 90) (layer B.SilkS)
-    (effects (font (size 1 1) (thickness 0.2)) (justify mirror))
-  )
   (gr_text BAT- (at 6.25 -2.65 270) (layer B.SilkS)
     (effects (font (size 1.2 1.2) (thickness 0.25)) (justify mirror))
@@
   (segment (start 4.8375 -19.4125) (end 1.2 -19.4125) (width 0.15) (layer F.Cu) (net 3))
   (segment (start 4.85 -19.4) (end 4.8375 -19.4125) (width 0.15) (layer F.Cu) (net 3))
-  (segment (start 2.2 -17.6) (end 6.2125 -17.6) (width 0.15) (layer F.Cu) (net 3))
-  (segment (start 1.2 -18.6) (end 2.2 -17.6) (width 0.15) (layer F.Cu) (net 3))
-  (segment (start 1.2 -19.4125) (end 1.2 -18.6) (width 0.15) (layer F.Cu) (net 3))
-  (segment (start 6.2125 -17.6) (end 7.6125 -19) (width 0.15) (layer F.Cu) (net 3))
   (segment (start 7.6125 -19) (end 7.6125 -16.2) (width 0.25) (layer F.Cu) (net 3))
   (segment (start 21.617878 -32.782122) (end 21.617878 -32.850022) (width 0.2) (layer F.Cu) (net 3))
@@
   (segment (start 22.657146 -36) (end 20.857133 -37.800013) (width 0.2) (layer B.Cu) (net 3))
   (segment (start 20.557134 -38.524276) (end 20.557134 -38.100012) (width 0.2) (layer F.Cu) (net 3))
+  (segment (start 2.1 -17.4) (end 6.0125 -17.4) (width 0.15) (layer F.Cu) (net 3))
+  (segment (start 6.0125 -17.4) (end 7.6125 -19) (width 0.15) (layer F.Cu) (net 3))
+  (segment (start 1.2 -18.3) (end 2.1 -17.4) (width 0.15) (layer F.Cu) (net 3))
+  (segment (start 1.2 -19.4125) (end 1.2 -18.3) (width 0.15) (layer F.Cu) (net 3))
   (via (at 29.769481 -32.168397) (size 0.6) (drill 0.3) (layers F.Cu B.Cu) (net 4))
   (segment (start 30.06948 -31.776816) (end 31.299987 -30.546309) (width 0.2) (layer F.Cu) (net 4))
@@
   (segment (start 24.4625 -27.2) (end 24.4625 -27.850504) (width 0.2) (layer F.Cu) (net 9) (status 10))
   (segment (start 3 -21.55) (end 2.75 -21.55) (width 0.15) (layer F.Cu) (net 9))
-  (segment (start 6.575736 -24.4) (end 7 -24.4) (width 0.15) (layer F.Cu) (net 9))
-  (segment (start 2.8 -21.85) (end 2.25 -22.4) (width 0.15) (layer F.Cu) (net 9))
-  (segment (start 3.294988 -24.4) (end 6.575736 -24.4) (width 0.15) (layer F.Cu) (net 9))
-  (segment (start 2.25 -22.4) (end 2.25 -23.355012) (width 0.15) (layer F.Cu) (net 9))
-  (segment (start 2.8 -21.55) (end 2.8 -21.85) (width 0.15) (layer F.Cu) (net 9))
-  (segment (start 2.25 -23.355012) (end 3.294988 -24.4) (width 0.15) (layer F.Cu) (net 9))
   (via (at 7 -24.4) (size 0.6) (drill 0.3) (layers F.Cu B.Cu) (net 9))
   (segment (start 22.499977 -17.394278) (end 18.969999 -13.864299) (width 0.2) (layer F.Cu) (net 9))
@@
   (via (at 10.817543 -24.067697) (size 0.6) (drill 0.3) (layers F.Cu B.Cu) (net 9))
   (segment (start 11.241807 -24.067697) (end 10.817543 -24.067697) (width 0.2) (layer F.Cu) (net 9))
+  (segment (start 6.575736 -24.4) (end 7 -24.4) (width 0.15) (layer F.Cu) (net 9))
+  (segment (start 2.8 -21.55) (end 2.8 -21.85) (width 0.15) (layer F.Cu) (net 9))
+  (segment (start 2.8 -21.85) (end 2.25 -22.4) (width 0.15) (layer F.Cu) (net 9))
+  (segment (start 2.25 -22.4) (end 2.25 -23.65) (width 0.15) (layer F.Cu) (net 9))
+  (segment (start 2.25 -23.65) (end 3 -24.4) (width 0.15) (layer F.Cu) (net 9))
+  (segment (start 3 -24.4) (end 6.575736 -24.4) (width 0.15) (layer F.Cu) (net 9))
   (segment (start 24.4625 -25.6) (end 23.8625 -26.2) (width 0.2) (layer F.Cu) (net 10) (status 10))
   (segment (start 24.06249 -28.00863) (end 24.06249 -28.016193) (width 0.2) (layer F.Cu) (net 10))
@@
   (segment (start 23.8625 -26.189692) (end 23.636395 -25.963587) (width 0.2) (layer F.Cu) (net 10))
   (via (at 7 -25.2) (size 0.6) (drill 0.3) (layers F.Cu B.Cu) (net 10))
-  (segment (start 3 -20.05) (end 1.935784 -20.05) (width 0.15) (layer F.Cu) (net 10))
-  (segment (start 1.710794 -20.27499) (end 0.739226 -20.27499) (width 0.15) (layer F.Cu) (net 10))
-  (segment (start 0.44999 -22.04999) (end 3.6 -25.2) (width 0.15) (layer F.Cu) (net 10))
-  (segment (start 0.44999 -20.564226) (end 0.44999 -22.04999) (width 0.15) (layer F.Cu) (net 10))
-  (segment (start 6.575736 -25.2) (end 7 -25.2) (width 0.15) (layer F.Cu) (net 10))
-  (segment (start 1.935784 -20.05) (end 1.710794 -20.27499) (width 0.15) (layer F.Cu) (net 10))
-  (segment (start 3.6 -25.2) (end 6.575736 -25.2) (width 0.15) (layer F.Cu) (net 10))
-  (segment (start 0.739226 -20.27499) (end 0.44999 -20.564226) (width 0.15) (layer F.Cu) (net 10))
   (segment (start 22.099967 -22.897448) (end 22.700012 -23.497493) (width 0.2) (layer F.Cu) (net 10))
   (segment (start 17.58 -13.04) (end 22.099967 -17.559967) (width 0.2) (layer F.Cu) (net 10))
@@
   (segment (start 14.424981 -24.824979) (end 10.898468 -24.824979) (width 0.2) (layer F.Cu) (net 10))
   (segment (start 16.741442 -24.899989) (end 14.499991 -24.899989) (width 0.2) (layer F.Cu) (net 10))
+  (segment (start 0.44999 -20.564226) (end 0.44999 -22.34498) (width 0.15) (layer F.Cu) (net 10))
+  (segment (start 1.710794 -20.27499) (end 0.739226 -20.27499) (width 0.15) (layer F.Cu) (net 10))
+  (segment (start 1.935784 -20.05) (end 1.710794 -20.27499) (width 0.15) (layer F.Cu) (net 10))
+  (segment (start 0.739226 -20.27499) (end 0.44999 -20.564226) (width 0.15) (layer F.Cu) (net 10))
+  (segment (start 0.44999 -22.34498) (end 3.30501 -25.2) (width 0.15) (layer F.Cu) (net 10))
+  (segment (start 3 -20.05) (end 1.935784 -20.05) (width 0.15) (layer F.Cu) (net 10))
+  (segment (start 3.30501 -25.2) (end 6.575736 -25.2) (width 0.15) (layer F.Cu) (net 10))
+  (segment (start 6.575736 -25.2) (end 7 -25.2) (width 0.15) (layer F.Cu) (net 10))
   (via (at 20.324272 -50.324272) (size 0.6) (drill 0.3) (layers F.Cu B.Cu) (net 11))
   (segment (start 20.400012 -50.400012) (end 20.324272 -50.324272) (width 0.2) (layer F.Cu) (net 11))
