File: rev2final/oibus-mini-CCC.sch (KiCad schematic (older format))
At the start: 89 parts, among them J1 Conn_01x04_Female, J2 USB_B_Micro, J3 uavcan_5pins, J4 Conn_01x02_Female, P1 TC2030-MCP, Q1 DMG3415U-7, Q2 NMOS, Q3 NMOS, SW1 SW_Push, SW2 SW_Push, U1 AP2112K-3.3, U10 TPD3E001DRLR, U2 SAM-M8Q, U3 NINA-B311-00B, U4 MCP73831-2-OT, U5 MCP1624T, U6 SHT31-DIS-B, U7 TCAN330, U8 STM32F303CCTx, U9 DW01C-G, Y1 16M, Y2 32kHz

Commit message: generated final rev2 assembly files ready for PCBA
Parts:
- added C13: 100n, Capacitor_SMD:C_0603_1608Metric, symbol Device:C_Small
- BT1: LCSC C160352 -> C64658; MPN B2B-PH-SM4-TB(LF)(SN) -> C64658; MPN2 (none) -> PH-2AW; MPN3 (none) -> B2B-PH-SM4-TB(LF)(SN)
- H2: MPN PHF254TH2x6 -> A2541HWV-2x6P; MPN2 (none) -> PHF254TH2x6
- R8: value 430R -> 1k
- SW2: MPN (none) -> SKSCLCE010
Connections:
- net GND: now also C13.2
- net on_off: now also C13.1
Changed lines of the file:
@@
 P 8200 10550
 F 0 "R8" H 8270 10596 50  0000 L CNN
-F 1 "430R" H 8270 10505 50  0000 L CNN
+F 1 "1k" H 8270 10505 50  0000 L CNN
 F 2 "Resistor_SMD:R_0603_1608Metric" V 8130 10550 50  0001 C CNN
 F 3 "~" H 8200 10550 50  0001 C CNN
@@
 F 2 "lib_fp_global:OIBUS12_connector" H 13350 6500 50  0001 C CNN
 F 3 "" H 13350 6500 50  0001 C CNN
-F 4 "PHF254TH2x6" H 200 450 50  0001 C CNN "MPN"
+F 4 "PHF254TH2x6" H 200 450 50  0001 C CNN "MPN2"
+F 5 "A2541HWV-2x6P" H 13350 6500 50  0001 C CNN "MPN"
 	1    13350 6500
 	1    0    0    -1
@@
 F 2 "Connector_JST:JST_PH_S2B-PH-K_1x02_P2.00mm_Horizontal" V 1050 8760 50  0001 C CNN
 F 3 "~" V 1050 8760 50  0001 C CNN
-F 4 "C160352" H 0   0   50  0001 C CNN "LCSC"
-F 5 "B2B-PH-SM4-TB(LF)(SN)" H 0   0   50  0001 C CNN "MPN"
+F 4 "C64658" H 0   0   50  0001 C CNN "LCSC"
+F 5 "B2B-PH-SM4-TB(LF)(SN)" H 0   0   50  0001 C CNN "MPN3"
+F 6 "PH-2AW" H 1050 8700 50  0001 C CNN "MPN2"
+F 7 "C64658" H 1050 8700 50  0001 C CNN "MPN"
 	1    1050 8700
 	-1   0    0    -1
@@
 F 2 "Button_Switch_SMD:SW_SPST_EVQP7C" H 10250 2600 50  0001 C CNN
 F 3 "~" H 10250 2600 50  0001 C CNN
+F 4 "SKSCLCE010" H 10250 2400 50  0001 C CNN "MPN"
 	1    10250 2400
 	1    0    0    -1
@@
 on_off
 Wire Wire Line
-	9700 2400 10050 2400
-Wire Wire Line
-	10450 2400 10650 2400
+	9700 2400 9900 2400
+Wire Wire Line
+	10450 2400 10500 2400
 Wire Wire Line
 	10650 2400 10650 2500
@@
 Wire Wire Line
 	13950 3700 14750 3700
+$Comp
+L Device:C_Small C13
+U 1 1 5DEAD42F
+P 10250 2600
+F 0 "C13" V 10300 2450 50  0000 C CNN
+F 1 "100n" V 10300 2750 50  0000 C CNN
+F 2 "Capacitor_SMD:C_0603_1608Metric" H 10250 2600 50  0001 C CNN
+F 3 "~" H 10250 2600 50  0001 C CNN
+F 4 "" H -2000 500 50  0001 C CNN "MPN"
+	1    10250 2600
+	0    -1   -1   0
+$EndComp
+Wire Wire Line
+	10350 2600 10500 2600
+Wire Wire Line
+	10500 2600 10500 2400
+Connection ~ 10500 2400
+Wire Wire Line
+	10500 2400 10650 2400
+Wire Wire Line
+	10150 2600 9900 2600
+Wire Wire Line
+	9900 2600 9900 2400
+Connection ~ 9900 2400
+Wire Wire Line
+	9900 2400 10050 2400
 $EndSCHEMATC
