File: rev2final/oibus-mini-CCC.kicad_pcb (KiCad board)
At the start: 2 copper layers, 37 x 60 mm, 92 parts, among them J1 Conn_01x04_Female, J2 USB_B_Micro, J3 uavcan_5pins, P1 TC2030-MCP, Q1 DMG3415U-7, Q2 NMOS, Q3 NMOS, SW1 SW_Push, SW2 SW_Push, U1 AP2112K-3.3, U10 TPD3E001DRLR, U2 SAM-M8Q, U3 NINA-B311-00B, U4 MCP73831-2-OT, U5 MCP1624T, U6 SHT31-DIS-B, U7 TCAN330, U8 STM32F303CCTx, U9 DW01C-G, Y1 16M, Y2 32kHz

Commit message: Generated final Manufacturing BOM as ordered
Parts:
- C25, C26: value 22p -> 10p
- D5: value LED_blue -> LED_blue_side
- D6: value D_TVS_x2_AAC -> DNP
- H2: value OIBUS_12.1_CONN -> DNP
- J3: value uavcan_5pins -> DNP
- R14, R15, R16, R3: value 1k -> 1.2k
- R17: value 2k7 -> 2.7k
- R19, R20: value 60R -> DNP
- R2: value 10k -> 5.1k
- R8: value 1k -> DNP
- U7: value TCAN330 -> DNP
- renumbered NFC to J4
Connections:
- J2 pad 4: (no net) -> /ID
- U1 pad 4: (no net) -> Net-(U1-Pad4)
- U10 pad 4: (no net) -> Net-(U10-Pad4)
- U2 pad 12: (no net) -> Net-(U2-Pad12)
- U2 pad 19: (no net) -> Net-(U2-Pad19)
- U2 pad 8: (no net) -> Net-(U2-Pad8)
- U2 pad 9: (no net) -> Net-(U2-Pad9)
- U3 pad 1: (no net) -> Net-(U3-Pad1)
- U3 pad 13: (no net) -> Net-(U3-Pad13)
- U3 pad 18: (no net) -> Net-(U3-Pad18)
- U3 pad 2: (no net) -> Net-(U3-Pad2)
- U3 pad 24: (no net) -> Net-(U3-Pad24)
- U3 pad 25: (no net) -> Net-(U3-Pad25)
- U3 pad 27: (no net) -> Net-(U3-Pad27)
- U3 pad 3: (no net) -> Net-(U3-Pad3)
- U3 pad 32: (no net) -> Net-(U3-Pad32)
- U3 pad 33: (no net) -> Net-(U3-Pad33)
- U3 pad 34: (no net) -> Net-(U3-Pad34)
- U3 pad 35: (no net) -> Net-(U3-Pad35)
- U3 pad 36: (no net) -> Net-(U3-Pad36)
- U3 pad 37: (no net) -> Net-(U3-Pad37)
- U3 pad 38: (no net) -> Net-(U3-Pad38)
- U3 pad 39: (no net) -> Net-(U3-Pad39)
- U3 pad 4: (no net) -> Net-(U3-Pad4)
- U3 pad 40: (no net) -> Net-(U3-Pad40)
- U3 pad 41: (no net) -> Net-(U3-Pad41)
- U3 pad 42: (no net) -> Net-(U3-Pad42)
- U3 pad 43: (no net) -> Net-(U3-Pad43)
- U3 pad 44: (no net) -> Net-(U3-Pad44)
- U3 pad 45: (no net) -> Net-(U3-Pad45)
- U3 pad 46: (no net) -> Net-(U3-Pad46)
- U3 pad 47: (no net) -> Net-(U3-Pad47)
- U3 pad 48: (no net) -> Net-(U3-Pad48)
- U3 pad 49: (no net) -> Net-(U3-Pad49)
- U3 pad 5: (no net) -> Net-(U3-Pad5)
- U3 pad 50: (no net) -> Net-(U3-Pad50)
- U3 pad 51: (no net) -> Net-(U3-Pad51)
- U3 pad 52: (no net) -> Net-(U3-Pad52)
- U3 pad 7: (no net) -> Net-(U3-Pad7)
- U3 pad 8: (no net) -> Net-(U3-Pad8)
- U6 pad 3: (no net) -> /SHT_ALERT
- U6 pad 6: (no net) -> Net-(U6-Pad6)
- U9 pad 4: (no net) -> Net-(U9-Pad4)

Commit message: added final BOM with proven parts values; de-cluttered repository; generated HTML BOM
Parts:
- C2: value 47u 16V -> 33uF ±20% 25V
- R17: value 2.7k -> 1.5k
- R8: value DNP -> 2.7k
Changed lines of the file:
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@@
       (effects (font (size 0.8 0.8) (thickness 0.15)))
     )
-    (fp_text value "47u 16V" (at 0 3.7) (layer F.Fab)
+    (fp_text value "33uF ±20% 25V " (at 0 3.7) (layer F.Fab)
       (effects (font (size 1 1) (thickness 0.15)))
     )
@@
       (effects (font (size 0.8 0.8) (thickness 0.15)))
     )
-    (fp_text value DNP (at 0 1.43 90) (layer F.Fab)
+    (fp_text value 2.7k (at 0 1.43 90) (layer F.Fab)
       (effects (font (size 1 1) (thickness 0.15)))
     )
@@
       (effects (font (size 0.8 0.8) (thickness 0.15)))
     )
-    (fp_text value 2.7k (at 0 1.43 270) (layer F.Fab)
-      (effects (font (size 1 1) (thickness 0.15)))
-    )
+    (fp_text value 1.5k (at 0 1.43 270) (layer F.Fab)
+      (effects (font (size 1 1) (thickness 0.15)))
+    )
